File: hardware/PCB/_autosave-FABI_schematic.sch (KiCad schematic (older format))
At the start: 45 parts, among them J1 AudioJack3_Ground, J10 Conn_01x03_Male, J11 dispaly_connector_91601-304LF, J11_GND1 Conn_01x01_Male, J11_VDD1 Conn_01x01_Male, J11_data1 Conn_01x01_Male, J2 AudioJack3_Ground, J3 AudioJack3_Ground, J4 AudioJack3_Ground, J5 AudioJack3_Ground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

Commit message: PCB: buzzer Resistor & silkscreen updates
Signed-off-by: fussthalerandreas <fussthaler.andreas1997@gmail.com>
Parts:
- J9: RS https://at.rs-online.com/web/p/leiterplatten-header/2518272/ -> https://at.rs-online.com/web/p/leiterplatten-header/7457040/; RS-Nr 251-8272 -> 745-7040
- R8: value 150 -> 200; RS https://at.rs-online.com/web/p/widerstande-durchsteckmontage/1650319/ -> https://at.rs-online.com/web/p/widerstande-durchsteckmontage/6833281/; RS-Nr 165-0319 -> 683-3281
- R_8: value 150 -> 200; RS https://at.rs-online.com/web/p/smd-widerstande/9059679/ -> https://at.rs-online.com/web/p/smd-widerstande/8101741/; RS-Nr 905-9679 -> 810-1741
Changed lines of the file:
@@
 F 2 "Connector_PinHeader_2.54mm:PinHeader_2x05_P2.54mm_Vertical" H 7410 5010 50  0001 C CNN
 F 3 "~" H 7410 5010 50  0001 C CNN
-F 4 "https://at.rs-online.com/web/p/leiterplatten-header/2518272/" H 7410 5010 50  0001 C CNN "RS"
-F 5 "251-8272" H 7410 5010 50  0001 C CNN "RS-Nr"
+F 4 "https://at.rs-online.com/web/p/leiterplatten-header/7457040/" H 7410 5010 50  0001 C CNN "RS"
+F 5 "745-7040" H 7410 5010 50  0001 C CNN "RS-Nr"
 	1    7410 5010
 	1    0    0    -1
@@
 P 9060 4965
 F 0 "R8" V 9267 4965 50  0000 C CNN
-F 1 "150" V 9176 4965 50  0000 C CNN
+F 1 "200" V 9176 4965 50  0000 C CNN
 F 2 "Resistor_THT:R_Axial_DIN0204_L3.6mm_D1.6mm_P7.62mm_Horizontal" V 8990 4965 50  0001 C CNN
 F 3 "~" H 9060 4965 50  0001 C CNN
-F 4 "https://at.rs-online.com/web/p/widerstande-durchsteckmontage/1650319/" V 9060 4965 50  0001 C CNN "RS"
-F 5 "165-0319" V 9060 4965 50  0001 C CNN "RS-Nr"
+F 4 "https://at.rs-online.com/web/p/widerstande-durchsteckmontage/6833281/" V 9060 4965 50  0001 C CNN "RS"
+F 5 "683-3281" V 9060 4965 50  0001 C CNN "RS-Nr"
 	1    9060 4965
 	0    -1   -1   0
@@
 P 9060 5115
 F 0 "R_8" V 8945 5115 50  0000 C CNN
-F 1 "150" V 8854 5115 50  0000 C CNN
+F 1 "200" V 8854 5115 50  0000 C CNN
 F 2 "Resistor_SMD:R_0805_2012Metric_Pad1.20x1.40mm_HandSolder" V 8990 5115 50  0001 C CNN
 F 3 "~" H 9060 5115 50  0001 C CNN
-F 4 "https://at.rs-online.com/web/p/smd-widerstande/9059679/" V 9060 5115 50  0001 C CNN "RS"
-F 5 "905-9679" V 9060 5115 50  0001 C CNN "RS-Nr"
+F 4 "https://at.rs-online.com/web/p/smd-widerstande/8101741/" V 9060 5115 50  0001 C CNN "RS"
+F 5 "810-1741" V 9060 5115 50  0001 C CNN "RS-Nr"
 	1    9060 5115
 	0    -1   -1   0
