File: hardware/PCB/FABI_schematic.sch (KiCad schematic (older format))
At the start: 37 parts, among them J1 Cliff_68125, J10 Conn_01x03_Male, J11 Conn_01x04_Male, J11_disp1 Conn_01x04_Female, J2 Cliff_68125, J3 Cliff_68125, J4 Cliff_68125, J5 Cliff_68125, J6 Cliff_68125, J7 Cliff_68125, J8 Cliff_68125, J9 Conn_02x05_Odd_Even, U1 MPXV7007GP, U2 ProMicro

Commit message: JackPlug Footprint changed
Signed-off-by: fussthalerandreas <fussthaler.andreas1997@gmail.com>
Parts:
- J1, J2, J3, J4, J5, J6, J7, J8: footprint CLIFF_FC68125:CLIFF_FC68125 -> SamacSys_Parts:FC68125
Connections:
- net labels added: AddOn_Pin1, AddOn_Pin2, AddOn_Pin3, SCL, SDA
- no-connect marks 33 -> 25
Other:
- note removed: "SCL"
- note removed: "SDA"
Changed lines of the file:
@@
 NoConn ~ 3600 3150
 NoConn ~ 3600 3250
-NoConn ~ 3600 3350
-NoConn ~ 3600 3850
-NoConn ~ 3600 3950
-NoConn ~ 3600 4050
 NoConn ~ 3600 3050
 Wire Wire Line
@@
 NoConn ~ 2350 7150
 NoConn ~ 2350 7250
-Text GLabel 1850 3350 0    39   Input ~ 0
+Text GLabel 1850 3950 0    39   Input ~ 0
 1
-Text GLabel 1850 3450 0    39   Input ~ 0
+Text GLabel 1850 4050 0    39   Input ~ 0
 2
 Text GLabel 1850 3550 0    39   Input ~ 0
@@
 Text GLabel 1850 3850 0    39   Input ~ 0
 6
-Text GLabel 1850 3950 0    39   Input ~ 0
+Text GLabel 3600 3950 2    39   Input ~ 0
 7
-Text GLabel 1850 4050 0    39   Input ~ 0
+Text GLabel 3600 4050 2    39   Input ~ 0
 8
 Wire Wire Line
@@
 	1    0    0    -1
 $EndComp
-NoConn ~ 7000 4850
-NoConn ~ 7500 4850
-NoConn ~ 7000 4950
-NoConn ~ 7500 4950
-NoConn ~ 7000 5050
 $Comp
 L power:GND #PWR010
@@
 P 5650 4850
 F 0 "#PWR015" H 5650 4700 50  0001 C CNN
-F 1 "VCC" H 5665 5023 50  0000 C CNN
+F 1 "VCC" V 5665 4978 50  0000 L CNN
 F 2 "" H 5650 4850 50  0001 C CNN
 F 3 "" H 5650 4850 50  0001 C CNN
@@
 	-1   0    0    -1
 $EndComp
-Text Label 5650 4950 0    39   ~ 0
-NEOPIXEL
 Text Label 3600 3650 0    39   ~ 0
 MPX
@@
 Text Notes 2300 2200 0    39   ~ 0
 Arduino Pro Micro
-NoConn ~ 3600 3450
 Text Label 3600 3750 0    39   ~ 0
 NEOPIXEL
@@
 F 0 "J3" H 882 6775 50  0000 C CNN
 F 1 "Cliff_68125" H 882 6684 50  0000 C CNN
-F 2 "CLIFF_FC68125:CLIFF_FC68125" H 900 6450 50  0001 C CNN
+F 2 "SamacSys_Parts:FC68125" H 900 6450 50  0001 C CNN
 F 3 "~" H 900 6450 50  0001 C CNN
 	1    900  6450
@@
 F 0 "J4" H 882 7575 50  0000 C CNN
 F 1 "Cliff_68125" H 882 7484 50  0000 C CNN
-F 2 "CLIFF_FC68125:CLIFF_FC68125" H 900 7250 50  0001 C CNN
+F 2 "SamacSys_Parts:FC68125" H 900 7250 50  0001 C CNN
 F 3 "~" H 900 7250 50  0001 C CNN
 	1    900  7250
@@
 F 0 "J5" H 2132 5175 50  0000 C CNN
 F 1 "Cliff_68125" H 2132 5084 50  0000 C CNN
-F 2 "CLIFF_FC68125:CLIFF_FC68125" H 2150 4850 50  0001 C CNN
+F 2 "SamacSys_Parts:FC68125" H 2150 4850 50  0001 C CNN
 F 3 "~" H 2150 4850 50  0001 C CNN
 	1    2150 4850
@@
 F 0 "J6" H 2132 5975 50  0000 C CNN
 F 1 "Cliff_68125" H 2132 5884 50  0000 C CNN
-F 2 "CLIFF_FC68125:CLIFF_FC68125" H 2150 5650 50  0001 C CNN
+F 2 "SamacSys_Parts:FC68125" H 2150 5650 50  0001 C CNN
 F 3 "~" H 2150 5650 50  0001 C CNN
 	1    2150 5650
@@
 F 0 "J8" H 2132 7575 50  0000 C CNN
 F 1 "Cliff_68125" H 2132 7484 50  0000 C CNN
-F 2 "CLIFF_FC68125:CLIFF_FC68125" H 2150 7250 50  0001 C CNN
+F 2 "SamacSys_Parts:FC68125" H 2150 7250 50  0001 C CNN
 F 3 "~" H 2150 7250 50  0001 C CNN
 	1    2150 7250
@@
 F 0 "J1" H 882 5175 50  0000 C CNN
 F 1 "Cliff_68125" H 882 5084 50  0000 C CNN
-F 2 "CLIFF_FC68125:CLIFF_FC68125" H 900 4850 50  0001 C CNN
+F 2 "SamacSys_Parts:FC68125" H 900 4850 50  0001 C CNN
 F 3 "~" H 900 4850 50  0001 C CNN
 	1    900  4850
@@
 F 0 "J2" H 882 5975 50  0000 C CNN
 F 1 "Cliff_68125" H 882 5884 50  0000 C CNN
-F 2 "CLIFF_FC68125:CLIFF_FC68125" H 900 5650 50  0001 C CNN
+F 2 "SamacSys_Parts:FC68125" H 900 5650 50  0001 C CNN
 F 3 "~" H 900 5650 50  0001 C CNN
 	1    900  5650
@@
 F 0 "J7" H 2132 6775 50  0000 C CNN
 F 1 "Cliff_68125" H 2132 6684 50  0000 C CNN
-F 2 "CLIFF_FC68125:CLIFF_FC68125" H 2150 6450 50  0001 C CNN
+F 2 "SamacSys_Parts:FC68125" H 2150 6450 50  0001 C CNN
 F 3 "~" H 2150 6450 50  0001 C CNN
 	1    2150 6450
@@
 $EndComp
 Text GLabel 8925 2950 0    39   Input ~ 0
-1
+SCL
 Text GLabel 8925 2625 0    39   Input ~ 0
-2
+SDA
 $Comp
 L power:GND #PWR020
@@
 	0    1    -1   0
 $EndComp
-Text Notes 8700 2975 0    39   ~ 0
-SCL
-Text Notes 8700 2650 0    39   ~ 0
-SDA
 Wire Wire Line
 	9800 3050 9800 2625
@@
 Text Notes 5305 6414 2    39   ~ 0
 SMD
+Text GLabel 3600 3350 2    39   Input ~ 0
+AddOn_Pin1
+Text GLabel 3600 3450 2    39   Input ~ 0
+AddOn_Pin2
+Text GLabel 3600 3850 2    39   Input ~ 0
+AddOn_Pin3
+Text GLabel 7000 4950 0    39   Input ~ 0
+AddOn_Pin3
+Text GLabel 7500 4850 2    39   Input ~ 0
+AddOn_Pin2
+Text GLabel 7000 4850 0    39   Input ~ 0
+AddOn_Pin1
+Text GLabel 1850 3350 0    39   Input ~ 0
+SCL
+Text GLabel 1850 3450 0    39   Input ~ 0
+SDA
+NoConn ~ 7500 4950
+NoConn ~ 7000 5050
+Text Label 5650 4950 0    39   ~ 0
+NEOPIXEL
 $EndSCHEMATC

Commit message: Pins changed and connected to AddOn
Signed-off-by: fussthalerandreas <fussthaler.andreas1997@gmail.com>
Connections:
- net labels added: Buzzer_Pin
- net labels removed: buzzer_pin
- wire segments 87 -> 86
Other:
- moved on the sheet: D11, D12
Changed lines of the file:
@@
 L Power_Protection:SP0504BAHT D12
 U 1 1 5F3C5FAA
-P 4200 4900
-F 0 "D12" H 4505 4946 50  0000 L CNN
-F 1 "SP0504BAHT" H 4250 4700 50  0000 L CNN
-F 2 "Package_TO_SOT_SMD:SOT-23-5" H 4500 4850 50  0001 L CNN
-F 3 "http://www.littelfuse.com/~/media/files/littelfuse/technical%20resources/documents/data%20sheets/sp05xxba.pdf" H 4325 5025 50  0001 C CNN
-	1    4200 4900
+P 4250 4900
+F 0 "D12" H 4555 4946 50  0000 L CNN
+F 1 "SP0504BAHT" H 4300 4700 50  0000 L CNN
+F 2 "Package_TO_SOT_SMD:SOT-23-5" H 4550 4850 50  0001 L CNN
+F 3 "http://www.littelfuse.com/~/media/files/littelfuse/technical%20resources/documents/data%20sheets/sp05xxba.pdf" H 4375 5025 50  0001 C CNN
+	1    4250 4900
 	1    0    0    -1
 $EndComp
@@
 L Power_Protection:SP0504BAHT D11
 U 1 1 5F3C6CE7
-P 3550 4900
-F 0 "D11" H 3855 4946 50  0000 L CNN
-F 1 "SP0504BAHT" H 3600 4700 50  0000 L CNN
-F 2 "Package_TO_SOT_SMD:SOT-23-5" H 3850 4850 50  0001 L CNN
-F 3 "http://www.littelfuse.com/~/media/files/littelfuse/technical%20resources/documents/data%20sheets/sp05xxba.pdf" H 3675 5025 50  0001 C CNN
-	1    3550 4900
-	1    0    0    -1
-$EndComp
-Text GLabel 3750 4700 1    39   Input ~ 0
+P 3600 4900
+F 0 "D11" H 3905 4946 50  0000 L CNN
+F 1 "SP0504BAHT" H 3650 4700 50  0000 L CNN
+F 2 "Package_TO_SOT_SMD:SOT-23-5" H 3900 4850 50  0001 L CNN
+F 3 "http://www.littelfuse.com/~/media/files/littelfuse/technical%20resources/documents/data%20sheets/sp05xxba.pdf" H 3725 5025 50  0001 C CNN
+	1    3600 4900
+	1    0    0    -1
+$EndComp
+Text GLabel 3800 4700 1    39   Input ~ 0
 1
-Text GLabel 3450 4700 1    39   Input ~ 0
+Text GLabel 3500 4700 1    39   Input ~ 0
 2
-Text GLabel 3550 4700 1    39   Input ~ 0
+Text GLabel 3600 4700 1    39   Input ~ 0
 3
-Text GLabel 3650 4700 1    39   Input ~ 0
+Text GLabel 3700 4700 1    39   Input ~ 0
 4
-Text GLabel 4200 4700 1    39   Input ~ 0
+Text GLabel 4250 4700 1    39   Input ~ 0
 5
-Text GLabel 4100 4700 1    39   Input ~ 0
+Text GLabel 4150 4700 1    39   Input ~ 0
 6
-Text GLabel 4400 4700 1    39   Input ~ 0
+Text GLabel 4450 4700 1    39   Input ~ 0
 7
-Text GLabel 4300 4700 1    39   Input ~ 0
+Text GLabel 4350 4700 1    39   Input ~ 0
 8
 $Comp
 L power:GND #PWR026
 U 1 1 5F3C927A
-P 3550 5100
-F 0 "#PWR026" H 3550 4850 50  0001 C CNN
-F 1 "GND" V 3555 4972 50  0000 R CNN
-F 2 "" H 3550 5100 50  0001 C CNN
-F 3 "" H 3550 5100 50  0001 C CNN
-	1    3550 5100
+P 3600 5100
+F 0 "#PWR026" H 3600 4850 50  0001 C CNN
+F 1 "GND" V 3605 4972 50  0000 R CNN
+F 2 "" H 3600 5100 50  0001 C CNN
+F 3 "" H 3600 5100 50  0001 C CNN
+	1    3600 5100
 	-1   0    0    -1
 $EndComp
@@
 L power:GND #PWR027
 U 1 1 5F3C9749
-P 4200 5100
-F 0 "#PWR027" H 4200 4850 50  0001 C CNN
-F 1 "GND" V 4205 4972 50  0000 R CNN
-F 2 "" H 4200 5100 50  0001 C CNN
-F 3 "" H 4200 5100 50  0001 C CNN
-	1    4200 5100
+P 4250 5100
+F 0 "#PWR027" H 4250 4850 50  0001 C CNN
+F 1 "GND" V 4255 4972 50  0000 R CNN
+F 2 "" H 4250 5100 50  0001 C CNN
+F 3 "" H 4250 5100 50  0001 C CNN
+	1    4250 5100
 	-1   0    0    -1
 $EndComp
@@
 Wire Notes Line
 	3300 4400 4850 4400
-Text GLabel 3650 3550 2    39   Input ~ 0
-buzzer_pin
+Text GLabel 3600 3550 2    39   Input ~ 0
+Buzzer_Pin
 Text GLabel 9325 4625 0    39   Input ~ 0
-buzzer_pin
+Buzzer_Pin
 $Comp
 L power:GND #PWR0101
@@
 Wire Wire Line
 	9325 4625 9425 4625
-Wire Wire Line
-	3600 3550 3650 3550
 Wire Notes Line
 	10100 4400 10100 5550

Commit message: Display positioning: adding adapted PinSocket to enable soldering and pluggin in of the display, 3D Models adapted
Signed-off-by: fussthalerandreas <fussthaler.andreas1997@gmail.com>
Parts:
- removed J11: Conn_01x04_Male, Connector:display, symbol Connector:Conn_01x04_Male
- added J11_display_socket1: 91601-304LF, SamacSys_Parts:91601304LF, symbol SamacSys_Parts:91601-304LF
- added R11: 10k, Resistor_SMD:R_0805_2012Metric_Pad1.20x1.40mm_HandSolder, symbol Device:R
- added R12: 18k, Resistor_SMD:R_0805_2012Metric_Pad1.20x1.40mm_HandSolder, symbol Device:R
- added R13: 10k, Resistor_THT:R_Axial_DIN0204_L3.6mm_D1.6mm_P7.62mm_Horizontal, symbol Device:R
- added R14: 18k, Resistor_THT:R_Axial_DIN0204_L3.6mm_D1.6mm_P7.62mm_Horizontal, symbol Device:R
- J11_disp1: footprint Connector_PinSocket_2.54mm:PinSocket_1x04_P2.54mm_Vertical -> FABI_customLibs:OLED_display_091
Connections:
- net labels added: ESP_AddOn_Pin1, VDD
- wire segments 86 -> 109
- no-connect marks 25 -> 20
Other:
- note added: "Arduino->ESP Connector - Reversed Pin"
- note added: "RAW: unregulated voltage input for the Pro Micro\nVCC: regulated voltage, 5V at 500mA\n"
- moved on the sheet: R10, R7, R8, R9

Commit message: Signed-off-by: fussthalerandreas <fussthaler.andreas1997@gmail.com>
Parts:
- removed J11_disp1: Conn_01x04_Female, FABI_customLibs:OLED_display_091, symbol Connector:Conn_01x04_Female
- removed J11_display_socket1: 91601-304LF, SamacSys_Parts:91601304LF, symbol SamacSys_Parts:91601-304LF
- added J11: dispaly_connector_91601-304LF, FABI_customLibs:91601304LF, symbol FABI_customLib:dispaly_connector_91601-304LF
Connections:
- wire segments 109 -> 101
- no-connect marks 20 -> 24
Other:
- moved on the sheet: R10, R7, R8, R9
Changed lines of the file:
@@
 L power:VCC #PWR019
 U 1 1 6027585C
-P 8750 3350
-F 0 "#PWR019" H 8750 3200 50  0001 C CNN
-F 1 "VCC" V 8765 3523 50  0000 C CNN
-F 2 "" H 8750 3350 50  0001 C CNN
-F 3 "" H 8750 3350 50  0001 C CNN
-	1    8750 3350
+P 8020 3240
+F 0 "#PWR019" H 8020 3090 50  0001 C CNN
+F 1 "VCC" V 8035 3413 50  0000 C CNN
+F 2 "" H 8020 3240 50  0001 C CNN
+F 3 "" H 8020 3240 50  0001 C CNN
+	1    8020 3240
 	0    -1   -1   0
 $EndComp
-Text GLabel 8720 3050 0    39   Input ~ 0
+Text GLabel 7990 2940 0    39   Input ~ 0
 SCL
-Text GLabel 8725 2700 0    39   Input ~ 0
+Text GLabel 7995 2590 0    39   Input ~ 0
 SDA
 $Comp
 L power:GND #PWR020
 U 1 1 60275866
-P 8750 3450
-F 0 "#PWR020" H 8750 3200 50  0001 C CNN
-F 1 "GND" V 8755 3322 50  0000 R CNN
-F 2 "" H 8750 3450 50  0001 C CNN
-F 3 "" H 8750 3450 50  0001 C CNN
-	1    8750 3450
+P 8020 3340
+F 0 "#PWR020" H 8020 3090 50  0001 C CNN
+F 1 "GND" V 8025 3212 50  0000 R CNN
+F 2 "" H 8020 3340 50  0001 C CNN
+F 3 "" H 8020 3340 50  0001 C CNN
+	1    8020 3340
 	0    1    -1   0
 $EndComp
@@
 L Device:R R8
 U 1 1 6031DA69
-P 9100 2850
-F 0 "R8" H 9030 2896 50  0000 R CNN
-F 1 "4.7k" H 9030 2805 50  0000 R CNN
-F 2 "Resistor_THT:R_Axial_DIN0204_L3.6mm_D1.6mm_P7.62mm_Horizontal" V 9030 2850 50  0001 C CNN
-F 3 "~" H 9100 2850 50  0001 C CNN
-	1    9100 2850
+P 8370 2740
+F 0 "R8" H 8300 2786 50  0000 R CNN
+F 1 "4.7k" H 8300 2695 50  0000 R CNN
+F 2 "Resistor_THT:R_Axial_DIN0204_L3.6mm_D1.6mm_P7.62mm_Horizontal" V 8300 2740 50  0001 C CNN
+F 3 "~" H 8370 2740 50  0001 C CNN
+	1    8370 2740
 	1    0    0    -1
 $EndComp
@@
 L Device:R R7
 U 1 1 6031DA63
-P 9000 3200
-F 0 "R7" H 8930 3246 50  0000 R CNN
-F 1 "4.7k" H 8930 3155 50  0000 R CNN
-F 2 "Resistor_THT:R_Axial_DIN0204_L3.6mm_D1.6mm_P7.62mm_Horizontal" V 8930 3200 50  0001 C CNN
-F 3 "~" H 9000 3200 50  0001 C CNN
-	1    9000 3200
-	1    0    0    -1
-$EndComp
-Wire Wire Line
-	8750 3350 9000 3350
-Connection ~ 9100 2700
-Wire Wire Line
-	9100 2700 8725 2700
-$Comp
-L Connector:Conn_01x04_Female J11_disp1
-U 1 1 6027586C
-P 10190 2800
-F 0 "J11_disp1" H 10218 2776 50  0000 L CNN
-F 1 "Conn_01x04_Female" H 10218 2685 50  0000 L CNN
-F 2 "FABI_customLibs:OLED_display_091" H 10190 2800 50  0001 C CNN
-F 3 "~" H 10190 2800 50  0001 C CNN
-	1    10190 2800
-	1    0    0    -1
-$EndComp
+P 8270 3090
+F 0 "R7" H 8200 3136 50  0000 R CNN
+F 1 "4.7k" H 8200 3045 50  0000 R CNN
+F 2 "Resistor_THT:R_Axial_DIN0204_L3.6mm_D1.6mm_P7.62mm_Horizontal" V 8200 3090 50  0001 C CNN
+F 3 "~" H 8270 3090 50  0001 C CNN
+	1    8270 3090
+	1    0    0    -1
+$EndComp
+Wire Wire Line
+	8020 3240 8270 3240
+Connection ~ 8370 2590
+Wire Wire Line
+	8370 2590 7995 2590
 $Comp
 L Device:R R9
 U 1 1 602F7E46
-P 9400 3200
-F 0 "R9" H 9330 3246 50  0000 R CNN
-F 1 "4.7k" H 9330 3155 50  0000 R CNN
-F 2 "Resistor_SMD:R_0805_2012Metric_Pad1.20x1.40mm_HandSolder" V 9330 3200 50  0001 C CNN
-F 3 "~" H 9400 3200 50  0001 C CNN
-	1    9400 3200
+P 8670 3090
+F 0 "R9" H 8600 3136 50  0000 R CNN
+F 1 "4.7k" H 8600 3045 50  0000 R CNN
+F 2 "Resistor_SMD:R_0805_2012Metric_Pad1.20x1.40mm_HandSolder" V 8600 3090 50  0001 C CNN
+F 3 "~" H 8670 3090 50  0001 C CNN
+	1    8670 3090
 	1    0    0    -1
 $EndComp
@@
 Text Notes 9140 5210 0    39   ~ 0
 SMD
-Text Notes 9440 3240 1    39   ~ 0
-SMD
-Wire Wire Line
-	9500 2700 9100 2700
+Text Notes 8710 3130 1    39   ~ 0
+SMD
+Wire Wire Line
+	8770 2590 8370 2590
 $Comp
 L Device:R R10
 U 1 1 602F9FD4
-P 9500 2850
-F 0 "R10" H 9430 2896 50  0000 R CNN
-F 1 "4.7k" H 9430 2805 50  0000 R CNN
-F 2 "Resistor_SMD:R_0805_2012Metric_Pad1.20x1.40mm_HandSolder" V 9430 2850 50  0001 C CNN
-F 3 "~" H 9500 2850 50  0001 C CNN
-	1    9500 2850
-	1    0    0    -1
-$EndComp
-Text Notes 9535 2910 1    39   ~ 0
+P 8770 2740
+F 0 "R10" H 8700 2786 50  0000 R CNN
+F 1 "4.7k" H 8700 2695 50  0000 R CNN
+F 2 "Resistor_SMD:R_0805_2012Metric_Pad1.20x1.40mm_HandSolder" V 8700 2740 50  0001 C CNN
+F 3 "~" H 8770 2740 50  0001 C CNN
+	1    8770 2740
+	1    0    0    -1
+$EndComp
+Text Notes 8805 2800 1    39   ~ 0
 SMD
 Text Notes 5305 6414 2    39   ~ 0
@@
 Text Notes 3230 2430 0    39   ~ 0
 RAW:   unregulated voltage input for the Pro Micro\nVCC:   regulated voltage, 5V at 500mA\n
-$Comp
-L SamacSys_Parts:91601-304LF J11_display_socket1
-U 1 1 6025E661
-P 10190 3450
-F 0 "J11_display_socket1" H 10590 3715 50  0000 C CNN
-F 1 "91601-304LF" H 10590 3624 50  0000 C CNN
-F 2 "SamacSys_Parts:91601304LF" H 10840 3550 50  0001 L CNN
-F 3 "http://www.mouser.com/datasheet/2/18/91601-1289404.pdf" H 10840 3450 50  0001 L CNN
-F 4 "Dubox 2.54mm, Board to Board Connector, PCB Mounted Receptacle, Vertical , Surface Mount, Dual Entry ,Single row , 4 Positions, 2.54mm (0.100in) Pitch" H 10840 3350 50  0001 L CNN "Description"
-F 5 "8" H 10840 3250 50  0001 L CNN "Height"
-F 6 "649-91601-304LF" H 10840 3150 50  0001 L CNN "Mouser Part Number"
-F 7 "https://www.mouser.com/Search/Refine.aspx?Keyword=649-91601-304LF" H 10840 3050 50  0001 L CNN "Mouser Price/Stock"
-F 8 "Amphenol" H 10840 2950 50  0001 L CNN "Manufacturer_Name"
-F 9 "91601-304LF" H 10840 2850 50  0001 L CNN "Manufacturer_Part_Number"
-	1    10190 3450
-	1    0    0    -1
-$EndComp
-Wire Wire Line
-	9500 2700 9820 2700
-Connection ~ 9500 2700
-Wire Wire Line
-	9100 3000 9100 3350
-Connection ~ 9100 3350
-Wire Wire Line
-	9100 3350 9400 3350
-Wire Wire Line
-	9500 3000 9500 3350
-Connection ~ 9500 3350
-Connection ~ 9000 3350
-Wire Wire Line
-	9000 3350 9100 3350
-Connection ~ 9400 3350
-Wire Wire Line
-	9400 3350 9500 3350
-Wire Wire Line
-	8720 3050 9000 3050
-Connection ~ 9000 3050
-Wire Wire Line
-	9000 3050 9400 3050
-Connection ~ 9400 3050
-Wire Wire Line
-	9400 3050 9600 3050
-Wire Wire Line
-	9600 3050 9600 2800
-Wire Wire Line
-	9600 2800 9990 2800
-Wire Wire Line
-	9670 3350 9670 2900
-Wire Wire Line
-	9670 2900 9990 2900
-Wire Wire Line
-	9500 3350 9670 3350
-Wire Wire Line
-	9740 3000 9990 3000
-Wire Wire Line
-	9740 3000 9740 3450
-Wire Wire Line
-	9740 3450 8750 3450
-Wire Wire Line
-	9740 3450 10190 3450
-Connection ~ 9740 3450
-Wire Wire Line
-	9670 3350 9670 3550
-Wire Wire Line
-	9670 3550 10190 3550
-Connection ~ 9670 3350
-Wire Wire Line
-	9600 3050 9600 3650
-Wire Wire Line
-	9600 3650 10190 3650
-Connection ~ 9600 3050
-Wire Wire Line
-	9820 2700 9820 3750
-Wire Wire Line
-	9820 3750 10190 3750
-Connection ~ 9820 2700
-Wire Wire Line
-	9820 2700 9990 2700
+Wire Wire Line
+	8770 2590 9090 2590
+Connection ~ 8770 2590
+Wire Wire Line
+	8370 2890 8370 3240
+Connection ~ 8370 3240
+Wire Wire Line
+	8370 3240 8670 3240
+Wire Wire Line
+	8770 2890 8770 3240
+Connection ~ 8770 3240
+Connection ~ 8270 3240
+Wire Wire Line
+	8270 3240 8370 3240
+Connection ~ 8670 3240
+Wire Wire Line
+	8670 3240 8770 3240
+Wire Wire Line
+	7990 2940 8270 2940
+Connection ~ 8270 2940
+Wire Wire Line
+	8270 2940 8670 2940
+Connection ~ 8670 2940
+Wire Wire Line
+	8670 2940 8870 2940
+Wire Wire Line
+	8770 3240 8940 3240
+Wire Wire Line
+	8940 3240 8940 3440
+Wire Wire Line
+	8870 2940 8870 3540
+Wire Wire Line
+	9090 2590 9090 3640
+NoConn ~ 9990 3540
+NoConn ~ 9990 3640
+NoConn ~ 9990 3440
+NoConn ~ 9990 3340
+$Comp
+L FABI_customLib:dispaly_connector_91601-304LF J11
+U 1 1 603EB941
+P 9190 3340
+F 0 "J11" H 9590 3605 50  0000 C CNN
+F 1 "dispaly_connector_91601-304LF" H 9590 3514 50  0000 C CNN
+F 2 "FABI_customLibs:91601304LF" H 10390 3390 50  0001 L CNN
+F 3 "http://www.mouser.com/datasheet/2/18/91601-1289404.pdf" H 10390 3290 50  0001 L CNN
+F 4 "Dubox 2.54mm, Board to Board Connector, PCB Mounted Receptacle, Vertical , Surface Mount, Dual Entry ,Single row , 4 Positions, 2.54mm (0.100in) Pitch" H 10390 3190 50  0001 L CNN "Description"
+F 5 "8" H 10390 3090 50  0001 L CNN "Height"
+F 6 "649-91601-304LF" H 10390 2990 50  0001 L CNN "Mouser Part Number"
+F 7 "https://www.mouser.com/Search/Refine.aspx?Keyword=649-91601-304LF" H 10390 2890 50  0001 L CNN "Mouser Price/Stock"
+F 8 "Amphenol" H 9390 2790 50  0001 L CNN "Manufacturer_Name"
+F 9 "91601-304LF" H 9390 2690 50  0001 L CNN "Manufacturer_Part_Number"
+	1    9190 3340
+	1    0    0    -1
+$EndComp
+Wire Wire Line
+	8020 3340 9190 3340
+Wire Wire Line
+	8940 3440 9190 3440
+Wire Wire Line
+	8870 3540 9190 3540
+Wire Wire Line
+	9090 3640 9190 3640
 $EndSCHEMATC

Commit message: routed the PCB, adapted all components, ready for review
Signed-off-by: fussthalerandreas <fussthaler.andreas1997@gmail.com>
Parts:
- R3, R4: footprint Resistor_SMD:R_0805_2012Metric_Pad1.15x1.40mm_HandSolder -> Resistor_SMD:R_0805_2012Metric_Pad1.20x1.40mm_HandSolder
- U1: footprint MPXV7007:MPXV7007GP -> MPXV7007GP:MPXV7007GP
Connections:
- net 1: now also U2.12 (D9/A9(PB5)); no longer U2.11 (D8/A8(PB4))
- net 2: now also U2.11 (D8/A8(PB4)); no longer U2.12 (D9/A9(PB5))
- net 3: now also U2.10 (D7(PE6)); no longer U2.7 (D4/A6(PD4))
- net 4: now also U2.9 (D6/A7(PD7)); no longer U2.8 (D5(PC6))
- net 5: now also U2.8 (D5(PC6)); no longer U2.9 (D6/A7(PD7))
- net 6: now also U2.18 (D19/A1(PF6)); no longer U2.10 (D7(PE6))
- net Buzzer_Pin: now also U2.7 (D4/A6(PD4)); no longer U2.18 (D19/A1(PF6))
- no-connect marks 24 -> 20
Changed lines of the file:
@@
 Sheet 1 1
 Title "FABI PCB for 8 jack plugs (ESP32 addon board conn)"
-Date "2020-08-15"
+Date "2021-02-11"
 Rev ""
 Comp "AsTeRICS Foundation"
@@
 NoConn ~ 2350 7150
 NoConn ~ 2350 7250
-Text GLabel 1850 3950 0    39   Input ~ 0
-1
-Text GLabel 1850 4050 0    39   Input ~ 0
-2
-Text GLabel 1850 3550 0    39   Input ~ 0
-3
-Text GLabel 1850 3650 0    39   Input ~ 0
-4
-Text GLabel 1850 3750 0    39   Input ~ 0
-5
-Text GLabel 1850 3850 0    39   Input ~ 0
-6
 Text GLabel 3600 3950 2    39   Input ~ 0
 7
-Text GLabel 3600 4050 2    39   Input ~ 0
-8
 Wire Wire Line
 	1850 3250 1850 3150
@@
 F 0 "R4" H 3620 6746 50  0000 L CNN
 F 1 "18k" H 3620 6655 50  0000 L CNN
-F 2 "Resistor_SMD:R_0805_2012Metric_Pad1.15x1.40mm_HandSolder" V 3480 6700 50  0001 C CNN
+F 2 "Resistor_SMD:R_0805_2012Metric_Pad1.20x1.40mm_HandSolder" V 3480 6700 50  0001 C CNN
 F 3 "~" H 3550 6700 50  0001 C CNN
 	1    3550 6700
@@
 F 0 "R3" H 3620 6346 50  0000 L CNN
 F 1 "10k" H 3620 6255 50  0000 L CNN
-F 2 "Resistor_SMD:R_0805_2012Metric_Pad1.15x1.40mm_HandSolder" V 3480 6300 50  0001 C CNN
+F 2 "Resistor_SMD:R_0805_2012Metric_Pad1.20x1.40mm_HandSolder" V 3480 6300 50  0001 C CNN
 F 3 "~" H 3550 6300 50  0001 C CNN
 	1    3550 6300
@@
 Wire Notes Line
 	3300 4400 4850 4400
-Text GLabel 3600 3550 2    39   Input ~ 0
-Buzzer_Pin
 Text GLabel 9325 4625 0    39   Input ~ 0
 Buzzer_Pin
@@
 F 0 "U1" H 5920 6546 50  0000 R CNN
 F 1 "MPXV7007GP" H 6250 6100 50  0000 R CNN
-F 2 "MPXV7007:MPXV7007GP" H 5850 6150 50  0001 C CNN
+F 2 "MPXV7007GP:MPXV7007GP" H 5850 6150 50  0001 C CNN
 F 3 "http://www.nxp.com/files/sensors/doc/data_sheet/MPXA6115A.pdf" H 6350 7100 50  0001 C CNN
 	1    6350 6500
@@
 Text Notes 9140 5210 0    39   ~ 0
 SMD
-Text Notes 8710 3130 1    39   ~ 0
+Text Notes 8700 3150 1    39   ~ 0
 SMD
 Wire Wire Line
@@
 Text Label 5650 4950 0    39   ~ 0
 NEOPIXEL
-$Comp
-L ProMicro:ProMicro U2
-U 1 1 601F96F3
-P 2700 3500
-F 0 "U2" H 2725 4275 50  0000 C CNN
-F 1 "ProMicro" H 2725 4184 50  0000 C CNN
-F 2 "ProMicro:ProMicro" H 2250 4150 50  0001 C CNN
-F 3 "" H 2250 4150 50  0001 C CNN
-	1    2700 3500
-	1    0    0    -1
-$EndComp
 Connection ~ 1850 3150
 $Comp
@@
 Wire Wire Line
 	9090 2590 9090 3640
-NoConn ~ 9990 3540
-NoConn ~ 9990 3640
-NoConn ~ 9990 3440
-NoConn ~ 9990 3340
+Wire Wire Line
+	8020 3340 9190 3340
+Wire Wire Line
+	9090 3640 9190 3640
+Text GLabel 1850 3750 0    39   Input ~ 0
+4
+Text GLabel 1850 3650 0    39   Input ~ 0
+5
+Text GLabel 1850 3950 0    39   Input ~ 0
+2
+Text GLabel 1850 4050 0    39   Input ~ 0
+1
+Text GLabel 1850 3850 0    39   Input ~ 0
+3
+Text GLabel 1850 3550 0    39   Input ~ 0
+Buzzer_Pin
+$Comp
+L ProMicro:ProMicro U2
+U 1 1 601F96F3
+P 2700 3500
+F 0 "U2" H 2725 4275 50  0000 C CNN
+F 1 "ProMicro" H 2725 4184 50  0000 C CNN
+F 2 "ProMicro:ProMicro" H 2250 4150 50  0001 C CNN
+F 3 "" H 2250 4150 50  0001 C CNN
+	1    2700 3500
+	1    0    0    -1
+$EndComp
+Wire Wire Line
+	9190 3440 8940 3440
+Wire Wire Line
+	9190 3540 8870 3540
 $Comp
 L FABI_customLib:dispaly_connector_91601-304LF J11
@@
 	1    0    0    -1
 $EndComp
-Wire Wire Line
-	8020 3340 9190 3340
-Wire Wire Line
-	8940 3440 9190 3440
-Wire Wire Line
-	8870 3540 9190 3540
-Wire Wire Line
-	9090 3640 9190 3640
+Text GLabel 3600 4050 2    39   Input ~ 0
+8
+Text GLabel 3600 3550 2    39   Input ~ 0
+6
 $EndSCHEMATC
