File: hardware/FABI_schematic.kicad_sch (KiCad schematic)
At the start: 40 parts, among them J11 009159005551906, J11_GND1 Conn_01x01_Male, J11_VDD1 Conn_01x01_Male, J11_data1 Conn_01x01_Male, J12 Conn_01x04_Socket, J2 display_connector_91601-304LF, Q1 BSS806, U1 D5V0F4U6SO, U2 SC0918 (PicoW), U3 TSOP4838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

Commit message: Fixed some messed up labels (imports from EAGLE); cleaned up unused libs
Parts:
- U1: footprint Package_TO_SOT_SMD:SC-74-6_1.55x2.9mm_P0.95mm -> Package_TO_SOT_SMD:SOT-23-6
Other:
- sheet Audio Amp ports: added pam8302_in, pam8302_sd; removed audio_out, audio_sd

Commit message: Added new Pico2W footprint to allow SMD headers (broader pads).
Parts:
- U2: footprint Module_RaspberryPi_Pico:RaspberryPi_Pico_W_SMD -> Module_RaspberryPi_Pico:RaspberryPi_Pico_W_SMD_header
Changed lines of the file:
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@@
 			)
 		)
-		(property "Footprint" "Module_RaspberryPi_Pico:RaspberryPi_Pico_W_SMD"
+		(property "Footprint" "Module_RaspberryPi_Pico:RaspberryPi_Pico_W_SMD_header"
 			(at 55.88 120.65 0)
 			(effects
